File: Peacock_Eagle/peacock3.sch (EAGLE design)
At the start: 111 parts, among them Q1 16M

Commit message: update
Parts:
- removed C45: 100uF, resistor:CPOL-USE5-6
- removed L3: (no value), resistor:L-USTJ5-U1
- U$1: device SparkFun-PowerIC:V_REG_LD1117VXX -> chikashilib:V_REG_LD1117VXX
Connections:
- removed net VDD: ADC1.VDD, ADC2.VDD, ADC3.VDD, ADC4.VDD, ADC5.VDD, C36.1, C37.1, C38.1, C39.1, C40.1
- net +3V3: now also U$1.SUP; no longer U$1.OUT
- net +5V: now also ADC1.VDD, ADC2.VDD, ADC3.VDD, ADC4.VDD, ADC5.VDD, ATMEGA32U2.UVCC, C36.1, C37.1, C38.1, C39.1, C40.1, L1.1, LCD.2, R4.2, R6.1, R8.2; no longer L3.1
- net GND: no longer C45.-
- net VCC: no longer ATMEGA32U2.UVCC, C45.+, L1.1, L3.2, LCD.2, R4.2, R6.1, R8.2
Other:
- moved on the sheet: ADC1, ADC2, ADC3, ADC4, ADC5, ATMEGA32U2, BUTTONS, C1, C10, C11, C12, C13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
