File: Peacock_Eagle/peacock3.sch (EAGLE design)
At the start: 100 parts, among them Q1 16M

Commit message: schemtic fixed
Parts:
- removed SENSOR1, SENSOR10, SENSOR11, SENSOR12, SENSOR13, SENSOR14, SENSOR15, SENSOR16, SENSOR17, SENSOR18, SENSOR19, SENSOR2, SENSOR20, SENSOR21, SENSOR22, SENSOR23, SENSOR24, SENSOR25, SENSOR26, SENSOR27, SENSOR28, SENSOR29, SENSOR3, SENSOR30, SENSOR31, SENSOR32, SENSOR33, SENSOR34, SENSOR35, SENSOR4, SENSOR5, SENSOR6, SENSOR7, SENSOR8, SENSOR9: (no value), pinhead:PINHD-1X3
- removed USB: (no value), SparkFun-Connectors:M04PTH
- added C45: 100uF, resistor:CPOL-USE5-6
- added C46: 1uF, resistor:C-USC1210
- added C47: 0.1uF, resistor:C-USC1210
- added C48: 10uF, resistor:C-USC1210
- added H1, H2, H3, H4: MOUNT-HOLE3.0, holes:MOUNT-HOLE3.0
- added JP1, JP10, JP11, JP12, JP13, JP14, JP15, JP16, JP17, JP18, JP19, JP2, JP20, JP21, JP22, JP23, JP24, JP25, JP26, JP27, JP28, JP29, JP3, JP30, JP31, JP32, JP33, JP34, JP35, JP4, JP5, JP6, JP7, JP8, JP9: (no value), SparkFun-Connectors:M03PTH
- added JP36: USB-B, SparkFun-Connectors:USBPTH
- added L2: 80R, resistor:L-US0207/12
- added L3: (no value), resistor:L-USTJ5-U1
- added U$1: V_REG_LD1117VXX, SparkFun-PowerIC:V_REG_LD1117VXX
- C1, C2: value 22pF -> 10uF; device resistor:C-EU050-024X044 -> resistor:C-USC1210
- C12, C13, C21, C29: value 0.1uF -> 10uF
- C36, C38, C39, C40, C42: value 10uF -> 0.1uF
- C41: value 10uF -> 100uF; device resistor:C-USC1210 -> resistor:CPOL-USE5-6
- C43: value 100uF -> 22pF; device resistor:CPOL-USE5-6 -> resistor:C-EU050-024X044
- C44: value 0.1uF -> 22pF; device resistor:C-USC1210 -> resistor:C-EU050-024X044
Connections:
- removed net N$18: R1.1, USB.2
- removed net N$37: SENSOR9.1
- removed net N$39: ADC2.CH3
- removed net N$40: SENSOR11.1
- removed net N$44: ADC3.CH5
- removed net N$47: SENSOR16.1
- removed net N$48: ADC3.CH3
- removed net N$49: SENSOR18.1
- removed net N$53: ADC4.CH5
- removed net N$56: SENSOR23.1
- removed net N$57: ADC4.CH3
- removed net N$58: SENSOR25.1
- removed net N$62: ADC5.CH5
- removed net N$65: SENSOR30.1
- removed net N$66: ADC5.CH3
- removed net N$67: SENSOR32.1
- new net N$29: ADC3.CH5, JP16.1
- new net N$30: ADC3.CH3, JP18.1
- new net N$32: ADC4.CH5, JP23.1
- new net N$33: ADC4.CH3, JP25.1
- new net N$34: ADC5.CH5, JP30.1
- net +3V3: now also C48.1, U$1.OUT
- net +5V: now also C1.1, C12.1, C13.1, C2.1, C21.1, C29.1, C47.1, JP1.3, JP10.3, JP11.3, JP12.3, JP13.3, JP14.3, JP15.3, JP16.3, JP17.3, JP18.3, JP19.3, JP2.3, JP20.3, JP21.3, JP22.3, JP23.3, JP24.3, JP25.3, JP26.3, JP27.3, JP28.3, JP29.3, JP3.3, JP30.3, JP31.3, JP32.3, JP33.3, JP34.3, JP35.3, JP4.3, JP5.3, JP6.3, JP7.3, JP8.3, JP9.3, L3.1, U$1.IN; no longer C36.1, C38.1, C39.1, C40.1, C41.1, C42.1, SENSOR1.3, SENSOR10.3, SENSOR11.3, SENSOR12.3, SENSOR13.3, SENSOR14.3, SENSOR15.3, SENSOR16.3, SENSOR17.3, SENSOR18.3, SENSOR19.3, SENSOR2.3, SENSOR20.3, SENSOR21.3, SENSOR22.3, SENSOR23.3, SENSOR24.3, SENSOR25.3, SENSOR26.3, SENSOR27.3, SENSOR28.3, SENSOR29.3, SENSOR3.3, SENSOR30.3, SENSOR31.3, SENSOR32.3, SENSOR33.3, SENSOR34.3, SENSOR35.3, SENSOR4.3, SENSOR5.3, SENSOR6.3, SENSOR7.3, SENSOR8.3, SENSOR9.3
- net AGND: now also ADC1.CH7, ADC1.DGND, ADC2.CH7, ADC2.DGND, ADC3.CH7, ADC3.DGND, ADC4.CH7, ADC4.DGND, ADC5.CH7, ADC5.DGND, C1.2, C2.2, C47.2, C48.2, JP1.2, JP10.2, JP11.2, JP12.2, JP13.2, JP14.2, JP15.2, JP16.2, JP17.2, JP18.2, JP19.2, JP2.2, JP20.2, JP21.2, JP22.2, JP23.2, JP24.2, JP25.2, JP26.2, JP27.2, JP28.2, JP29.2, JP3.2, JP30.2, JP31.2, JP32.2, JP33.2, JP34.2, JP35.2, JP4.2, JP5.2, JP6.2, JP7.2, JP8.2, JP9.2, L2.2, U$1.GND; no longer C41.2, C42.2, SENSOR1.2, SENSOR10.2, SENSOR11.2, SENSOR12.2, SENSOR13.2, SENSOR14.2, SENSOR15.2, SENSOR16.2, SENSOR17.2, SENSOR18.2, SENSOR19.2, SENSOR2.2, SENSOR20.2, SENSOR21.2, SENSOR22.2, SENSOR23.2, SENSOR24.2, SENSOR25.2, SENSOR26.2, SENSOR27.2, SENSOR28.2, SENSOR29.2, SENSOR3.2, SENSOR30.2, SENSOR31.2, SENSOR32.2, SENSOR33.2, SENSOR34.2, SENSOR35.2, SENSOR4.2, SENSOR5.2, SENSOR6.2, SENSOR7.2, SENSOR8.2, SENSOR9.2
- net CS5: now also ADC5.~CS
- net GND: now also C41.-, C42.2, C45.-, C46.2, JP36.GND, L2.1; no longer C43.-, C44.2, USB.3
- net MISO: now also ADC4.DOUT
- net N$1: now also C43.1, C44.1; no longer C1.1, C2.1
- net N$10: now also JP36.VBUS, L1.2; no longer ADC1.DGND, ADC2.DGND, ADC3.DGND, ADC4.DGND, ADC5.DGND
- net N$11: now also ADC1.CH5, JP2.1; no longer SENSOR2.1
- net N$12: now also JP1.1; no longer SENSOR1.1
- net N$13: now also ADC2.CH3, JP11.1; no longer ADC1.CH5
- net N$14: now also ATMEGA32U2.D+; no longer ATMEGA32U2.D-
- net N$15: now also JP36.D+; no longer USB.1
- net N$16: now also JP36.D-, R1.1; no longer ATMEGA32U2.D+, R1.2
- net N$17: now also JP3.1; no longer SENSOR3.1
- net N$2: now also JP8.1; no longer SENSOR8.1
- net N$25: now also JP10.1; no longer SENSOR10.1
- net N$28: now also ATMEGA32U2.UCAP, C46.1; no longer L1.2, USB.4
- net N$3: now also ADC1.CH3, JP4.1; no longer SENSOR4.1
- net N$35: now also ADC5.CH3, JP32.1; no longer ADC1.CH3
- net N$36: now also JP12.1; no longer SENSOR12.1
- net N$38: now also JP5.1; no longer SENSOR5.1
- net N$4: now also JP7.1; no longer SENSOR7.1
- net N$41: now also JP14.1; no longer SENSOR14.1
- net N$42: now also JP13.1; no longer SENSOR13.1
- net N$43: now also JP15.1; no longer SENSOR15.1
- net N$45: now also JP17.1; no longer SENSOR17.1
- net N$46: now also JP19.1; no longer SENSOR19.1
- net N$5: now also JP6.1; no longer SENSOR6.1
- net N$50: now also JP21.1; no longer SENSOR21.1
- net N$51: now also JP20.1; no longer SENSOR20.1
- net N$52: now also JP22.1; no longer SENSOR22.1
- net N$54: now also JP24.1; no longer SENSOR24.1
- net N$55: now also JP26.1; no longer SENSOR26.1
- net N$59: now also JP28.1; no longer SENSOR28.1
- net N$6: now also JP9.1
- net N$60: now also JP27.1; no longer SENSOR27.1
- net N$61: now also JP29.1; no longer SENSOR29.1
- net N$63: now also JP31.1; no longer SENSOR31.1
- net N$64: now also JP33.1; no longer SENSOR33.1
- net N$68: now also JP35.1; no longer SENSOR35.1
- net N$69: now also JP34.1; no longer SENSOR34.1
- net N$7: now also ATMEGA32U2.D-, R1.2; no longer ADC1.CH7, ADC2.CH7, ADC3.CH7, ADC4.CH7, ADC5.CH7
- net N$8: now also C44.2; no longer C2.2
- net N$9: now also C43.2; no longer C1.2
- net VCC: now also C41.+, C42.1, C45.+, L3.2; no longer C43.+, C44.1
- net VDD: now also C36.1, C38.1, C39.1, C40.1; no longer C12.1, C13.1, C21.1, C29.1
Other:
- moved on the sheet: C1, C10, C11, C12, C13, C14, C15, C16, C17, C18, C19, C2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

Commit message: update
Parts:
- removed L2: 80R, resistor:L-US0207/12
Connections:
- removed net AGND: ADC1.AGND, ADC1.CH7, ADC1.DGND, ADC2.AGND, ADC2.CH7, ADC2.DGND, ADC3.AGND, ADC3.CH7, ADC3.DGND, ADC4.AGND, ADC4.CH7, ADC4.DGND, ADC5.AGND, ADC5.CH7, ADC5.DGND, C1.2, C10.2, C11.2, C12.2, C13.2, C14.2, C15.2, C16.2, C17.2, C18.2, C19.2, C2.2, C20.2, C21.2, C22.2, C23.2, C24.2, C25.2, C26.2, C27.2, C28.2, C29.2, C3.2, C30.2, C31.2, C32.2, C33.2, C34.2, C35.2, C36.2, C37.2, C38.2, C39.2, C4.2, C40.2, C47.2, C48.2, C5.2, C6.2, C7.2, C8.2, C9.2, JP1.2, JP10.2, JP11.2, JP12.2, JP13.2, JP14.2, JP15.2, JP16.2, JP17.2, JP18.2, JP19.2, JP2.2, JP20.2, JP21.2, JP22.2, JP23.2, JP24.2, JP25.2, JP26.2, JP27.2, JP28.2, JP29.2, JP3.2, JP30.2, JP31.2, JP32.2, JP33.2, JP34.2, JP35.2, JP4.2, JP5.2, JP6.2, JP7.2, JP8.2, JP9.2, L2.2, U$1.GND
- new net N$49: C21.2, JP21.2
- net GND: now also ADC1.AGND, ADC1.CH7, ADC1.DGND, ADC2.AGND, ADC2.CH7, ADC2.DGND, ADC3.AGND, ADC3.CH7, ADC3.DGND, ADC4.AGND, ADC4.CH7, ADC4.DGND, ADC5.AGND, ADC5.CH7, ADC5.DGND, C1.2, C10.2, C11.2, C12.2, C13.2, C14.2, C15.2, C16.2, C17.2, C18.2, C19.2, C2.2, C20.2, C22.2, C23.2, C24.2, C25.2, C26.2, C27.2, C28.2, C29.2, C3.2, C30.2, C31.2, C32.2, C33.2, C34.2, C35.2, C36.2, C37.2, C38.2, C39.2, C4.2, C40.2, C47.2, C48.2, C5.2, C6.2, C7.2, C8.2, C9.2, JP1.2, JP10.2, JP11.2, JP12.2, JP13.2, JP14.2, JP15.2, JP16.2, JP17.2, JP18.2, JP19.2, JP2.2, JP20.2, JP22.2, JP23.2, JP24.2, JP25.2, JP26.2, JP27.2, JP28.2, JP29.2, JP3.2, JP30.2, JP31.2, JP32.2, JP33.2, JP34.2, JP35.2, JP4.2, JP5.2, JP6.2, JP7.2, JP8.2, JP9.2, U$1.GND; no longer L2.1

Commit message: power update
Parts:
- removed C45: 100uF, resistor:CPOL-USE5-6
- removed L3: (no value), resistor:L-USTJ5-U1
Connections:
- removed net VCC: ATMEGA32U2.AVCC, ATMEGA32U2.UVCC, ATMEGA32U2.VCC, C41.+, C42.1, C45.+, L1.1, L3.2, LCD.2, R4.2, R6.1, R8.2
- removed net VDD: ADC1.VDD, ADC2.VDD, ADC3.VDD, ADC4.VDD, ADC5.VDD, C36.1, C37.1, C38.1, C39.1, C40.1
- net +5V: now also ADC1.VDD, ADC2.VDD, ADC3.VDD, ADC4.VDD, ADC5.VDD, ATMEGA32U2.AVCC, ATMEGA32U2.UVCC, ATMEGA32U2.VCC, C36.1, C37.1, C38.1, C39.1, C40.1, C41.+, C42.1, L1.1, LCD.2, R4.2, R6.1, R8.2; no longer L3.1
- net GND: no longer C45.-

Commit message: routing done
Parts:
- removed ADC1, ADC2, ADC3, ADC4, ADC5: MCP3208/DIP, mcp3208:MCP3208/DIP
- removed BUTTONS: (no value), SparkFun-Connectors:M05PTH
- removed H4: MOUNT-HOLE3.0, holes:MOUNT-HOLE3.0
- removed L1: 80R, resistor:L-US0207/12
- added JP37: (no value), SparkFun-Connectors:M04PTH
- added U$3, U$4, U$5, U$6, U$7: MCP3208I/SL, myLibrary:MCP3208I/SL
- C36, C37, C38, C39, C40: value 0.1uF -> 10uF
- U$1: device SparkFun-PowerIC:V_REG_LD1117VXX -> myLibrary:V_REG_LD1117VXX
- renumbered GND to GND_SOCKET, JUMPER to HWB, LCD to LCD_SOCKET
Connections:
- removed net CS1: ADC1.~CS, ATMEGA32U2.PB0(SS/PCINT0)
- removed net CS2: ADC2.~CS, ATMEGA32U2.PB4(T1/PCINT4)
- removed net CS3: ADC3.~CS, ATMEGA32U2.PB5(PCINT5)
- removed net CS4: ADC4.~CS, ATMEGA32U2.PB6(PCINT6)
- removed net CS5: ADC5.~CS, ATMEGA32U2.PB7(INT4/ICP1/CLKO)
- removed net N$10: JP36.VBUS, L1.2
- removed net N$21: ATMEGA32U2.PC4(PCINT10), BUTTONS.3
- removed net N$23: ATMEGA32U2.PC6(OC.1A/PCINT8), BUTTONS.1
- removed net N$31: ATMEGA32U2.PC7(INT4/ICP1/CLKO), LED1.A
- removed net N$49: C21.2, JP21.2
- new net N$39: ATMEGA32U2.PB0(SS/PCINT0), U$3.!CS
- new net N$40: ATMEGA32U2.PB7(INT4/ICP1/CLKO), U$7.!CS
- new net N$44: ATMEGA32U2.PB6(PCINT6), U$6.!CS
- new net N$47: ATMEGA32U2.PB4(T1/PCINT4), U$4.!CS
- new net N$48: ATMEGA32U2.PB5(PCINT5), U$5.!CS
- net +3V3: now also LED1.A, U$3.VREF, U$4.VREF, U$5.VREF, U$6.VREF, U$7.VREF; no longer ADC1.VREF, ADC2.VREF, ADC3.VREF, ADC4.VREF, ADC5.VREF
- net +5V: now also JP36.VBUS, U$3.VDD, U$4.VDD, U$5.VDD, U$6.VDD, U$7.VDD; no longer ADC1.VDD, ADC2.VDD, ADC3.VDD, ADC4.VDD, ADC5.VDD, L1.1
- net CLK: now also U$3.CLK, U$4.CLK, U$5.CLK, U$6.CLK, U$7.CLK; no longer ADC1.CLK, ADC2.CLK, ADC3.CLK, ADC4.CLK, ADC5.CLK
- net GND: now also ATMEGA32U2.UGND, C21.2, C43.1, C44.1, JP21.2, U$3.AGND, U$3.CH0, U$3.DGND, U$4.AGND, U$4.CH0, U$4.DGND, U$5.AGND, U$5.CH0, U$5.DGND, U$6.AGND, U$6.CH0, U$6.DGND, U$7.AGND, U$7.CH0, U$7.DGND; no longer ADC1.AGND, ADC1.CH7, ADC1.DGND, ADC2.AGND, ADC2.CH7, ADC2.DGND, ADC3.AGND, ADC3.CH7, ADC3.DGND, ADC4.AGND, ADC4.CH7, ADC4.DGND, ADC5.AGND, ADC5.CH7, ADC5.DGND
- net MISO: now also U$3.DOUT, U$4.DOUT, U$5.DOUT, U$6.DOUT, U$7.DOUT; no longer ADC1.DOUT, ADC2.DOUT, ADC3.DOUT, ADC4.DOUT, ADC5.DOUT
- net MOSI: now also U$3.DIN, U$4.DIN, U$5.DIN, U$6.DIN, U$7.DIN; no longer ADC1.DIN, ADC2.DIN, ADC3.DIN, ADC4.DIN, ADC5.DIN
- net N$1: now also ATMEGA32U2.PC4(PCINT10), JP37.1; no longer ATMEGA32U2.UGND, C43.1, C44.1
- net N$11: now also U$3.CH2; no longer ADC1.CH5
- net N$12: now also U$3.CH1; no longer ADC1.CH6
- net N$13: now also U$4.CH4; no longer ADC2.CH3
- net N$17: now also U$3.CH3; no longer ADC1.CH4
- net N$2: now also U$4.CH1; no longer ADC2.CH6
- net N$20: now also ATMEGA32U2.PC5(PCINT9/OC.1B), JP37.2; no longer ATMEGA32U2.PC2(PCINT11/AIN2), BUTTONS.4
- net N$22: now also ATMEGA32U2.PC6(OC.1A/PCINT8), JP37.4; no longer ATMEGA32U2.PC5(PCINT9/OC.1B), BUTTONS.2
- net N$25: now also U$4.CH3; no longer ADC2.CH4
- net N$26: now also JP37.3; no longer BUTTONS.5
- net N$29: now also U$5.CH2; no longer ADC3.CH5
- net N$3: now also U$3.CH4; no longer ADC1.CH3
- net N$30: now also U$5.CH4; no longer ADC3.CH3
- net N$32: now also U$6.CH2; no longer ADC4.CH5
- net N$33: now also U$6.CH4; no longer ADC4.CH3
- net N$34: now also U$7.CH2; no longer ADC5.CH5
- net N$35: now also U$7.CH4; no longer ADC5.CH3
- net N$36: now also U$4.CH5; no longer ADC2.CH2
- net N$38: now also U$3.CH5; no longer ADC1.CH2
- net N$4: now also U$3.CH7; no longer ADC1.CH0
- net N$41: now also U$4.CH7; no longer ADC2.CH0
- net N$42: now also U$4.CH6; no longer ADC2.CH1
- net N$43: now also U$5.CH1; no longer ADC3.CH6
- net N$45: now also U$5.CH3; no longer ADC3.CH4
- net N$46: now also U$5.CH5; no longer ADC3.CH2
- net N$5: now also U$3.CH6; no longer ADC1.CH1
- net N$50: now also U$5.CH7; no longer ADC3.CH0
- net N$51: now also U$5.CH6; no longer ADC3.CH1
- net N$52: now also U$6.CH1; no longer ADC4.CH6
- net N$54: now also U$6.CH3; no longer ADC4.CH4
- net N$55: now also U$6.CH5; no longer ADC4.CH2
- net N$59: now also U$6.CH7; no longer ADC4.CH0
- net N$6: now also U$4.CH2; no longer ADC2.CH5
- net N$60: now also U$6.CH6; no longer ADC4.CH1
- net N$61: now also U$7.CH1; no longer ADC5.CH6
- net N$63: now also U$7.CH3; no longer ADC5.CH4
- net N$64: now also U$7.CH5; no longer ADC5.CH2
- net N$68: now also U$7.CH7; no longer ADC5.CH0
- net N$69: now also U$7.CH6; no longer ADC5.CH1
Other:
- moved on the sheet: C36, C37, C38, C39, C40, LED1, R3
