File: Peacock_Eagle/peacock3.sch (EAGLE design)
At the start: 106 parts, among them Q1 16M

Commit message: peacock update
Parts:
- removed JP37: (no value), SparkFun-Connectors:M04PTH
- removed U$7: MCP3208I/SL, myLibrary:MCP3208I/SL
- added BUTTONS: (no value), SparkFun-Connectors:M06SIP
- added U$2: MCP3208, mcp3208:MCP3208
- U$3, U$4, U$5, U$6: value MCP3208I/SL -> MCP3208; device myLibrary:MCP3208I/SL -> mcp3208:MCP3208
Connections:
- removed net N$68: JP35.1, U$7.CH7
- removed net N$69: JP34.1, U$7.CH6
- new net N$62: JP32.1, U$2.CH4
- new net N$65: JP29.1, U$2.CH1
- new net N$66: JP26.1, U$3.CH5
- new net RESET: ATMEGA32U2.PC1(RESET/DW), BUTTONS.4, R4.1
- net +3V3: now also U$2.VREF; no longer U$7.VREF
- net +5V: now also U$2.VDD; no longer U$7.VDD
- net CLK: now also U$2.CLK; no longer U$7.CLK
- net GND: now also U$2.AGND, U$2.CH0, U$2.DGND; no longer U$7.AGND, U$7.CH0, U$7.DGND
- net MISO: now also U$2.DOUT; no longer U$7.DOUT
- net MOSI: now also U$2.DIN; no longer U$7.DIN
- net N$1: now also ATMEGA32U2.PC2(PCINT11/AIN2), BUTTONS.1; no longer ATMEGA32U2.PC4(PCINT10), JP37.1
- net N$11: now also JP20.1, U$4.CH6; no longer JP2.1, U$3.CH2
- net N$12: now also JP21.1, U$4.CH7; no longer JP1.1, U$3.CH1
- net N$13: now also JP1.1, U$6.CH1; no longer JP11.1, U$4.CH4
- net N$17: now also JP2.1, U$6.CH2; no longer JP3.1, U$3.CH3
- net N$2: now also JP15.1; no longer JP8.1
- net N$20: now also ATMEGA32U2.PC4(PCINT10), BUTTONS.2; no longer ATMEGA32U2.PC5(PCINT9/OC.1B), JP37.2
- net N$22: now also ATMEGA32U2.PC5(PCINT9/OC.1B), BUTTONS.3; no longer ATMEGA32U2.PC6(OC.1A/PCINT8), JP37.4
- net N$25: now also JP3.1, U$6.CH3; no longer JP10.1, U$4.CH3
- net N$26: now also ATMEGA32U2.PC6(OC.1A/PCINT8), BUTTONS.5; no longer ATMEGA32U2.PC1(RESET/DW), JP37.3, R4.1
- net N$29: now also JP4.1, U$6.CH4; no longer JP16.1, U$5.CH2
- net N$3: now also JP16.1, U$4.CH2; no longer JP4.1, U$3.CH4
- net N$30: now also JP5.1, U$6.CH5; no longer JP18.1, U$5.CH4
- net N$32: now also JP27.1, U$3.CH6; no longer JP23.1, U$6.CH2
- net N$33: now also JP28.1, U$3.CH7; no longer JP25.1, U$6.CH4
- net N$34: now also JP35.1, U$2.CH7; no longer JP30.1, U$7.CH2
- net N$35: now also JP34.1, U$2.CH6; no longer JP32.1, U$7.CH4
- net N$36: now also JP6.1, U$6.CH6; no longer JP12.1, U$4.CH5
- net N$38: now also JP7.1, U$6.CH7; no longer JP5.1, U$3.CH5
- net N$39: now also U$6.~CS; no longer U$3.!CS
- net N$4: now also JP17.1, U$4.CH3; no longer JP7.1, U$3.CH7
- net N$40: now also U$2.~CS; no longer U$7.!CS
- net N$41: now also U$5.CH7; no longer U$4.CH7
- net N$42: now also U$5.CH6; no longer U$4.CH6
- net N$43: now also JP12.1, U$5.CH5; no longer JP15.1, U$5.CH1
- net N$44: now also U$3.~CS; no longer U$6.!CS
- net N$45: now also JP11.1, U$5.CH4; no longer JP17.1, U$5.CH3
- net N$46: now also JP10.1, U$5.CH3; no longer JP19.1, U$5.CH5
- net N$47: now also U$5.~CS; no longer U$4.!CS
- net N$48: now also U$4.~CS; no longer U$5.!CS
- net N$5: now also JP18.1, U$4.CH4; no longer JP6.1, U$3.CH6
- net N$50: now also JP9.1, U$5.CH2; no longer JP21.1, U$5.CH7
- net N$51: now also JP8.1, U$5.CH1; no longer JP20.1, U$5.CH6
- net N$52: now also JP25.1, U$3.CH4; no longer JP22.1, U$6.CH1
- net N$54: now also U$3.CH3; no longer U$6.CH3
- net N$55: now also JP23.1, U$3.CH2; no longer JP26.1, U$6.CH5
- net N$59: now also ATMEGA32U2.PC7(INT4/ICP1/CLKO), BUTTONS.6; no longer JP28.1, U$6.CH7
- net N$6: now also JP19.1, U$4.CH5; no longer JP9.1, U$4.CH2
- net N$60: now also JP22.1, U$3.CH1; no longer JP27.1, U$6.CH6
- net N$61: now also JP33.1, U$2.CH5; no longer JP29.1, U$7.CH1
- net N$63: now also U$2.CH3; no longer U$7.CH3
- net N$64: now also JP30.1, U$2.CH2; no longer JP33.1, U$7.CH5
Other:
- moved on the sheet: C1, C10, C11, C12, C13, C14, C15, C16, C17, C18, C19, C2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

Commit message: LED fixed
Parts:
- removed BUTTONS, GND_SOCKET: (no value), SparkFun-Connectors:M06SIP
- added JP37, JP38: (no value), SparkFun-Connectors:M05PTH
Connections:
- net +3V3: no longer LED1.A
- net GND: now also JP38.1, JP38.2, JP38.3, JP38.4, JP38.5; no longer GND_SOCKET.1, GND_SOCKET.2, GND_SOCKET.3, GND_SOCKET.4, GND_SOCKET.5, GND_SOCKET.6
- net N$1: now also LED1.A; no longer BUTTONS.1
- net N$20: now also JP37.1; no longer BUTTONS.2
- net N$22: now also JP37.2; no longer BUTTONS.3
- net N$26: now also JP37.4; no longer BUTTONS.5
- net N$59: now also JP37.5; no longer BUTTONS.6
- net RESET: now also JP37.3; no longer BUTTONS.4
Changed lines of the file:
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@@
 <part name="HWB" library="SparkFun-Connectors" deviceset="M02" device="PTH"/>
 <part name="GND9" library="supply1" deviceset="GND" device=""/>
-<part name="GND_SOCKET" library="SparkFun-Connectors" deviceset="M06" device="SIP"/>
 <part name="GND7" library="supply1" deviceset="GND" device=""/>
 <part name="LCD_SOCKET" library="SparkFun-Connectors" deviceset="M12" device="PTH"/>
@@
 <part name="P+47" library="supply1" deviceset="+5V" device=""/>
 <part name="GND18" library="supply1" deviceset="GND" device=""/>
-<part name="+3V7" library="supply1" deviceset="+3V3" device=""/>
 <part name="GND53" library="supply1" deviceset="GND" device=""/>
 <part name="C36" library="resistor" deviceset="C-US" device="C1210" value="10uF"/>
@@
 <part name="U$5" library="mcp3208" deviceset="MCP3208" device=""/>
 <part name="U$6" library="mcp3208" deviceset="MCP3208" device=""/>
-<part name="BUTTONS" library="SparkFun-Connectors" deviceset="M06" device="SIP"/>
+<part name="JP37" library="SparkFun-Connectors" deviceset="M05" device="PTH"/>
+<part name="JP38" library="SparkFun-Connectors" deviceset="M05" device="PTH"/>
 </parts>
 <sheets>
@@
 <instance part="HWB" gate="G$1" x="104.14" y="167.64" rot="MR0"/>
 <instance part="GND9" gate="1" x="88.9" y="160.02"/>
-<instance part="GND_SOCKET" gate="G$1" x="106.68" y="297.18"/>
 <instance part="GND7" gate="1" x="114.3" y="287.02"/>
 <instance part="LCD_SOCKET" gate="G$1" x="134.62" y="210.82" rot="MR0"/>
@@
 </instance>
 <instance part="GND18" gate="1" x="-10.16" y="236.22"/>
-<instance part="+3V7" gate="G$1" x="66.04" y="302.26"/>
 <instance part="GND53" gate="1" x="223.52" y="226.06"/>
 <instance part="C36" gate="G$1" x="172.72" y="317.5"/>
@@
 <instance part="U$5" gate="G$1" x="190.5" y="259.08" rot="R180"/>
 <instance part="U$6" gate="G$1" x="190.5" y="330.2" rot="R180"/>
-<instance part="BUTTONS" gate="G$1" x="127" y="261.62" rot="R180"/>
+<instance part="JP37" gate="G$1" x="129.54" y="259.08" rot="R180"/>
+<instance part="JP38" gate="G$1" x="104.14" y="297.18"/>
 </instances>
 <busses>
@@
 <segment>
 <pinref part="GND7" gate="1" pin="GND"/>
-<wire x1="114.3" y1="304.8" x2="114.3" y2="302.26" width="0.1524" layer="91"/>
-<pinref part="GND_SOCKET" gate="G$1" pin="5"/>
 <wire x1="114.3" y1="302.26" x2="114.3" y2="299.72" width="0.1524" layer="91"/>
 <wire x1="114.3" y1="299.72" x2="114.3" y2="297.18" width="0.1524" layer="91"/>
@@
 <wire x1="114.3" y1="292.1" x2="114.3" y2="289.56" width="0.1524" layer="91"/>
 <wire x1="111.76" y1="302.26" x2="114.3" y2="302.26" width="0.1524" layer="91"/>
-<junction x="114.3" y="302.26"/>
-<pinref part="GND_SOCKET" gate="G$1" pin="4"/>
 <wire x1="111.76" y1="299.72" x2="114.3" y2="299.72" width="0.1524" layer="91"/>
 <junction x="114.3" y="299.72"/>
-<pinref part="GND_SOCKET" gate="G$1" pin="3"/>
 <wire x1="111.76" y1="297.18" x2="114.3" y2="297.18" width="0.1524" layer="91"/>
 <junction x="114.3" y="297.18"/>
-<pinref part="GND_SOCKET" gate="G$1" pin="2"/>
 <wire x1="111.76" y1="294.64" x2="114.3" y2="294.64" width="0.1524" layer="91"/>
 <junction x="114.3" y="294.64"/>
-<pinref part="GND_SOCKET" gate="G$1" pin="1"/>
 <wire x1="111.76" y1="292.1" x2="114.3" y2="292.1" width="0.1524" layer="91"/>
 <junction x="114.3" y="292.1"/>
-<pinref part="GND_SOCKET" gate="G$1" pin="6"/>
-<wire x1="111.76" y1="304.8" x2="114.3" y2="304.8" width="0.1524" layer="91"/>
+<pinref part="JP38" gate="G$1" pin="1"/>
+<pinref part="JP38" gate="G$1" pin="2"/>
+<pinref part="JP38" gate="G$1" pin="3"/>
+<pinref part="JP38" gate="G$1" pin="4"/>
+<pinref part="JP38" gate="G$1" pin="5"/>
 </segment>
 <segment>
@@
 <junction x="88.9" y="266.7"/>
 <wire x1="116.84" y1="266.7" x2="116.84" y2="259.08" width="0.1524" layer="91"/>
-<pinref part="BUTTONS" gate="G$1" pin="4"/>
 <wire x1="116.84" y1="259.08" x2="121.92" y2="259.08" width="0.1524" layer="91"/>
+<pinref part="JP37" gate="G$1" pin="3"/>
 </segment>
 </net>
@@
 <wire x1="76.2" y1="185.42" x2="71.12" y2="185.42" width="0.1524" layer="91"/>
 <junction x="76.2" y="185.42"/>
-</segment>
-<segment>
-<pinref part="LED1" gate="G$1" pin="A"/>
-<pinref part="+3V7" gate="G$1" pin="+3V3"/>
 </segment>
 <segment>
@@
 </segment>
 </net>
-<net name="N$1" class="0">
-<segment>
-<pinref part="ATMEGA32U2" gate="G$1" pin="PC2(PCINT11/AIN2)"/>
-<wire x1="88.9" y1="264.16" x2="106.68" y2="264.16" width="0.1524" layer="91"/>
-<wire x1="106.68" y1="264.16" x2="106.68" y2="269.24" width="0.1524" layer="91"/>
-<pinref part="BUTTONS" gate="G$1" pin="1"/>
-<wire x1="106.68" y1="269.24" x2="121.92" y2="269.24" width="0.1524" layer="91"/>
-<wire x1="121.92" y1="269.24" x2="121.92" y2="266.7" width="0.1524" layer="91"/>
-</segment>
-</net>
 <net name="N$20" class="0">
 <segment>
-<pinref part="BUTTONS" gate="G$1" pin="2"/>
 <wire x1="121.92" y1="264.16" x2="109.22" y2="264.16" width="0.1524" layer="91"/>
 <wire x1="109.22" y1="264.16" x2="109.22" y2="261.62" width="0.1524" layer="91"/>
 <pinref part="ATMEGA32U2" gate="G$1" pin="PC4(PCINT10)"/>
 <wire x1="109.22" y1="261.62" x2="88.9" y2="261.62" width="0.1524" layer="91"/>
+<pinref part="JP37" gate="G$1" pin="1"/>
 </segment>
 </net>
@@
 <wire x1="88.9" y1="259.08" x2="111.76" y2="259.08" width="0.1524" layer="91"/>
 <wire x1="111.76" y1="259.08" x2="111.76" y2="261.62" width="0.1524" layer="91"/>
-<pinref part="BUTTONS" gate="G$1" pin="3"/>
 <wire x1="111.76" y1="261.62" x2="121.92" y2="261.62" width="0.1524" layer="91"/>
+<pinref part="JP37" gate="G$1" pin="2"/>
 </segment>
 </net>
 <net name="N$26" class="0">
 <segment>
-<pinref part="BUTTONS" gate="G$1" pin="5"/>
 <pinref part="ATMEGA32U2" gate="G$1" pin="PC6(OC.1A/PCINT8)"/>
 <wire x1="121.92" y1="256.54" x2="88.9" y2="256.54" width="0.1524" layer="91"/>
+<pinref part="JP37" gate="G$1" pin="4"/>
 </segment>
 </net>
 <net name="N$59" class="0">
 <segment>
-<pinref part="BUTTONS" gate="G$1" pin="6"/>
 <pinref part="ATMEGA32U2" gate="G$1" pin="PC7(INT4/ICP1/CLKO)"/>
 <wire x1="121.92" y1="254" x2="88.9" y2="254" width="0.1524" layer="91"/>
-</segment>
-</net>
+<pinref part="JP37" gate="G$1" pin="5"/>
+</segment>
+</net>
+<net name="N$1" class="0">
+<segment>
+<pinref part="LED1" gate="G$1" pin="A"/>
+<wire x1="66.04" y1="299.72" x2="93.98" y2="299.72" width="0.1524" layer="91"/>
+<wire x1="93.98" y1="299.72" x2="93.98" y2="264.16" width="0.1524" layer="91"/>
+<pinref part="ATMEGA32U2" gate="G$1" pin="PC2(PCINT11/AIN2)"/>
+<wire x1="93.98" y1="264.16" x2="88.9" y2="264.16" width="0.1524" layer="91"/>
+</segment>
+</net>
