File: Peacock_Eagle/peacock3.brd (EAGLE design)
At the start: 100.2 x 80 mm, 106 parts, among them Q1 16M

Commit message: peacock update
Parts:
- removed JP37: (no value), SparkFun-Connectors:1X04
- removed U$7: MCP3208I/SL, myLibrary:SO-16DW
- added BUTTONS: (no value), SparkFun-Connectors:1X06
- added U$2: MCP3208, mcp3208:SO16
- U$3, U$4, U$5, U$6: value MCP3208I/SL -> MCP3208; device myLibrary:SO-16DW -> mcp3208:SO16
- moved U$3 57.5 mm to (36.5, 36.0)
- moved U$6 56.7 mm to (93.5, 36.0)
- moved U$4 19.4 mm to (55.5, 36.0)
- moved U$5 18.9 mm to (74.8, 36.0)
- moved GND_SOCKET 2.50 mm to (2.54, 9.56)
- moved C41 2.00 mm to (73.7, 14.1)
Connections:
- removed net N$68: JP35.1, U$7.8
- removed net N$69: JP34.1, U$7.7
- new net N$62: JP32.1, U$2.5
- new net N$65: JP29.1, U$2.2
- new net N$66: JP26.1, U$3.6
- new net RESET: ATMEGA32U2.24, BUTTONS.4, R4.1
- net +3V3: now also U$2.15; no longer U$7.15
- net +5V: now also U$2.16; no longer U$7.16
- net CLK: now also U$2.13; no longer U$7.13
- net GND: now also U$2.1, U$2.14, U$2.9; no longer U$7.1, U$7.14, U$7.9
- net MISO: now also U$2.12; no longer U$7.12
- net MOSI: now also U$2.11; no longer U$7.11
- net N$1: now also ATMEGA32U2.5, BUTTONS.1; no longer ATMEGA32U2.26, JP37.1
- net N$11: now also JP20.1, U$4.7; no longer JP2.1, U$3.3
- net N$12: now also JP21.1, U$4.8; no longer JP1.1, U$3.2
- net N$13: now also JP1.1, U$6.2; no longer JP11.1, U$4.5
- net N$17: now also JP2.1, U$6.3; no longer JP3.1, U$3.4
- net N$2: now also JP15.1; no longer JP8.1
- net N$20: now also ATMEGA32U2.26, BUTTONS.2; no longer ATMEGA32U2.25, JP37.2
- net N$22: now also ATMEGA32U2.25, BUTTONS.3; no longer ATMEGA32U2.23, JP37.4
- net N$25: now also JP3.1, U$6.4; no longer JP10.1, U$4.4
- net N$26: now also ATMEGA32U2.23, BUTTONS.5; no longer ATMEGA32U2.24, JP37.3, R4.1
- net N$29: now also JP4.1, U$6.5; no longer JP16.1, U$5.3
- net N$3: now also JP16.1, U$4.3; no longer JP4.1, U$3.5
- net N$30: now also JP5.1, U$6.6; no longer JP18.1, U$5.5
- net N$32: now also JP27.1, U$3.7; no longer JP23.1, U$6.3
- net N$33: now also JP28.1, U$3.8; no longer JP25.1, U$6.5
- net N$34: now also JP35.1, U$2.8; no longer JP30.1, U$7.3
- net N$35: now also JP34.1, U$2.7; no longer JP32.1, U$7.5
- net N$36: now also JP6.1, U$6.7; no longer JP12.1, U$4.6
- net N$38: now also JP7.1, U$6.8; no longer JP5.1, U$3.6
- net N$39: now also U$6.10; no longer U$3.10
- net N$4: now also JP17.1, U$4.4; no longer JP7.1, U$3.8
- net N$40: now also U$2.10; no longer U$7.10
- net N$41: now also U$5.8; no longer U$4.8
- net N$42: now also U$5.7; no longer U$4.7
- net N$43: now also JP12.1, U$5.6; no longer JP15.1, U$5.2
- net N$44: now also U$3.10; no longer U$6.10
- net N$45: now also JP11.1, U$5.5; no longer JP17.1, U$5.4
- net N$46: now also JP10.1, U$5.4; no longer JP19.1, U$5.6
- net N$47: now also U$5.10; no longer U$4.10
- net N$48: now also U$4.10; no longer U$5.10
- net N$5: now also JP18.1, U$4.5; no longer JP6.1, U$3.7
- net N$50: now also JP9.1, U$5.3; no longer JP21.1, U$5.8
- net N$51: now also JP8.1, U$5.2; no longer JP20.1, U$5.7
- net N$52: now also JP25.1, U$3.5; no longer JP22.1, U$6.2
- net N$54: now also U$3.4; no longer U$6.4
- net N$55: now also JP23.1, U$3.3; no longer JP26.1, U$6.6
- net N$59: now also ATMEGA32U2.22, BUTTONS.6; no longer JP28.1, U$6.8
- net N$6: now also JP19.1, U$4.6; no longer JP9.1, U$4.3
- net N$60: now also JP22.1, U$3.2; no longer JP27.1, U$6.7
- net N$61: now also JP33.1, U$2.6; no longer JP29.1, U$7.2
- net N$63: now also U$2.4; no longer U$7.4
- net N$64: now also JP30.1, U$2.3; no longer JP33.1, U$7.6
Routing:
- net N$65: track 0.00 -> 40.3 mm
- net RESET: track 0.00 -> 37.0 mm
- net N$43: track 42.6 -> 16.0 mm
- net N$61: track 42.6 -> 16.9 mm
- net N$52: track 42.6 -> 17.2 mm
- net N$13: track 17.6 -> 39.8 mm
- net N$68: track 21.5 -> 0.00 mm
- net N$60: track 19.0 -> 40.5 mm
- net N$51: track 19.0 -> 40.4 mm
- net N$12: track 42.4 -> 22.1 mm
- net N$69: track 19.0 -> 0.00 mm
- net N$62: track 0.00 -> 18.9 mm
- net N$6: track 34.1 -> 15.8 mm
- net N$64: track 15.8 -> 33.5 mm
- net N$55: track 15.8 -> 32.8 mm
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Other:
- board size 100.2 x 80 mm -> 100 x 80 mm
- board text added: "Peacock III (ver.0.2) by C.Miyama"

Commit message: LED fixed
Parts:
- removed BUTTONS, GND_SOCKET: (no value), SparkFun-Connectors:1X06
- added JP37, JP38: (no value), SparkFun-Connectors:1X05
- moved C47 1.00 mm to (85.7, 3.44)
- moved C48 1.00 mm to (85.7, 8.53)
Connections:
- net +3V3: no longer LED1.A
- net GND: now also JP38.1, JP38.2, JP38.3, JP38.4, JP38.5; no longer GND_SOCKET.1, GND_SOCKET.2, GND_SOCKET.3, GND_SOCKET.4, GND_SOCKET.5, GND_SOCKET.6
- net N$1: now also LED1.A; no longer BUTTONS.1
- net N$20: now also JP37.1; no longer BUTTONS.2
- net N$22: now also JP37.2; no longer BUTTONS.3
- net N$26: now also JP37.4; no longer BUTTONS.5
- net N$59: now also JP37.5; no longer BUTTONS.6
- net RESET: now also JP37.3; no longer BUTTONS.4
Routing:
- net N$1: track 37.2 -> 63.8 mm, vias 2 -> 1
- net GND: track 905.6 -> 915.3 mm
- net +3V3: track 150.3 -> 144.8 mm
- net RESET: track 37.0 -> 38.6 mm
- net N$20: track 29.1 -> 30.6 mm
- net N$22: track 28.4 -> 29.8 mm
- net N$59: track 36.0 -> 34.6 mm
- net N$9: track 20.6 -> 19.8 mm
- net N$7: track 31.7 -> 31.1 mm
- net N$26: track 32.8 -> 32.3 mm

Commit message: draft of paper
Routing:
- net +5V: track 800.8 -> 791.7 mm
- net GND: track 915.3 -> 911.7 mm
- net N$27: track 25.6 -> 24.5 mm
